File: pcb/usb_dev_pmod.kicad_pcb (KiCad board)
At the start: 4 copper layers, 37.3 x 17.5 mm, 12 parts, among them J3 PMOD B, J5 DEV DEBUG, J6 AU-Y1007, U2 STUSB03E

Commit message: Fix labels.
Other:
- board text added: "D_OE_"
- board text added: "D_RCV"
- board text added: "D_VM"
- board text added: "D_VP"
- board text removed: "H_OE_"
- board text removed: "H_RCV"
- board text removed: "H_VM"
- board text removed: "H_VP"
