File: pcb/usb_host_pmod.kicad_pcb (KiCad board)
At the start: 4 copper layers, 37.3 x 17.8 mm, 13 parts, among them J1 PMOD A, J2 HOST DEBUG, J4 USB_A, U1 STUSB03E

Commit message: Fix labels.
Other:
- board text added: "H_OE_"
- board text added: "H_RCV"
- board text added: "H_VM"
- board text added: "H_VP"
- board text removed: "D_OE_"
- board text removed: "D_RCV"
- board text removed: "D_VM"
- board text removed: "D_VP"
