File: pcb/usb_pmod.kicad_pcb (KiCad board)
At the start: 4 copper layers, 37.3 x 40.4 mm, 25 parts, among them J1 PMOD A, J2 HOST DEBUG, J3 PMOD B, J4 USB_A, J5 DEV DEBUG, J6 AU-Y1007, U1 STUSB03E, U2 STUSB03E

Commit message: Fix labels.
Connections:
- J4 pad 1: (no net) -> /H_VBUS
Routing:
- net /H_VBUS: track 5.06 -> 34.2 mm
Changed lines of the file:
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@@
     (thickness 1.6)
     (drawings 34)
-    (tracks 285)
+    (tracks 291)
     (zones 0)
     (modules 25)
@@
     (add_net /H_VM)
     (add_net /H_VP)
+    (add_net /I2C_SCL)
+    (add_net /I2C_SDA)
+    (add_net "Net-(U1-Pad13)")
+    (add_net "Net-(U1-Pad16)")
   )
   (net_class Power ""
@@
     (pad 2 thru_hole circle (at 2.5 0 90) (size 1.6 1.6) (drill 0.92) (layers *.Cu *.Mask)
       (net 28 /H_DN))
-    (pad 1 thru_hole rect (at 0 0 90) (size 1.6 1.6) (drill 0.92) (layers *.Cu *.Mask))
+    (pad 1 thru_hole rect (at 0 0 90) (size 1.6 1.6) (drill 0.92) (layers *.Cu *.Mask)
+      (net 22 /H_VBUS))
     (pad 5 thru_hole circle (at -3.07 2.71 90) (size 3 3) (drill 2.3) (layers *.Cu *.Mask)
       (net 5 GND))
@@
   (gr_line (start 81.28 106.68) (end 81.28 93.472) (layer Edge.Cuts) (width 0.05))
   (gr_line (start 88.392 86.106) (end 83.566 86.106) (layer Edge.Cuts) (width 0.05))
-  (gr_text D_RCV (at 95.504 103.632 90) (layer F.SilkS)
+  (gr_text H_RCV (at 95.504 103.632 90) (layer F.SilkS)
     (effects (font (size 0.6 0.6) (thickness 0.1)))
   )
   (gr_line (start 118.618 83.82) (end 118.618 70.866) (layer Edge.Cuts) (width 0.05))
-  (gr_text H_OE_ (at 98.044 80.899 270) (layer F.SilkS)
+  (gr_text D_OE_ (at 98.044 80.899 270) (layer F.SilkS)
     (effects (font (size 0.6 0.6) (thickness 0.1)))
   )
-  (gr_text "H_VP\n" (at 93.091 80.645 270) (layer F.SilkS)
+  (gr_text "D_VP\n" (at 93.091 80.645 270) (layer F.SilkS)
     (effects (font (size 0.6 0.6) (thickness 0.1)))
   )
@@
     (effects (font (size 0.6 0.6) (thickness 0.1)))
   )
-  (gr_text H_RCV (at 95.504 80.899 270) (layer F.SilkS)
+  (gr_text D_RCV (at 95.504 80.899 270) (layer F.SilkS)
     (effects (font (size 0.6 0.6) (thickness 0.1)))
   )
-  (gr_text "H_VM\n" (at 90.551 80.645 270) (layer F.SilkS)
+  (gr_text "D_VM\n" (at 90.551 80.645 270) (layer F.SilkS)
     (effects (font (size 0.6 0.6) (thickness 0.1)))
   )
-  (gr_text "D_VM\n" (at 90.424 103.886 90) (layer F.SilkS)
+  (gr_text "H_VM\n" (at 90.424 103.886 90) (layer F.SilkS)
     (effects (font (size 0.6 0.6) (thickness 0.1)))
   )
-  (gr_text "D_VP\n" (at 92.964 103.886 90) (layer F.SilkS)
+  (gr_text "H_VP\n" (at 92.964 103.886 90) (layer F.SilkS)
     (effects (font (size 0.6 0.6) (thickness 0.1)))
   )
-  (gr_text D_OE_ (at 98.044 103.632 90) (layer F.SilkS)
+  (gr_text H_OE_ (at 98.044 103.632 90) (layer F.SilkS)
     (effects (font (size 0.6 0.6) (thickness 0.1)))
   )
@@
   (segment (start 104.492 75.028) (end 101.346 71.882) (width 0.0889) (layer F.Cu) (net 21))
   (segment (start 104.492 76.002) (end 104.492 75.028) (width 0.0889) (layer F.Cu) (net 21))
-  (segment (start 91.965 94.234) (end 92.7905 95.0595) (width 0.0889) (layer F.Cu) (net 22))
-  (segment (start 91.44 94.234) (end 91.965 94.234) (width 0.0889) (layer F.Cu) (net 22))
-  (segment (start 92.7905 95.0595) (end 92.7905 96.283) (width 0.0889) (layer F.Cu) (net 22))
-  (segment (start 92.198 96.8755) (end 92.198 98.1825) (width 0.0889) (layer F.Cu) (net 22))
-  (segment (start 92.7905 96.283) (end 92.198 96.8755) (width 0.0889) (layer F.Cu) (net 22))
+  (segment (start 91.44 94.234) (end 90.551 93.345) (width 0.127) (layer F.Cu) (net 22))
+  (segment (start 90.551 92.4687) (end 91.0717 91.948) (width 0.127) (layer F.Cu) (net 22))
+  (segment (start 90.551 93.345) (end 90.551 92.4687) (width 0.127) (layer F.Cu) (net 22))
+  (segment (start 91.0717 91.948) (end 92.583 91.948) (width 0.127) (layer F.Cu) (net 22))
+  (segment (start 92.583 91.948) (end 94.234 93.599) (width 0.127) (layer F.Cu) (net 22))
+  (segment (start 94.234 93.599) (end 105.791 93.599) (width 0.127) (layer F.Cu) (net 22))
+  (segment (start 105.791 93.599) (end 108.204 96.012) (width 0.127) (layer F.Cu) (net 22))
+  (segment (start 108.204 101.764) (end 106.426 103.542) (width 0.127) (layer F.Cu) (net 22))
+  (segment (start 108.204 96.012) (end 108.204 101.764) (width 0.127) (layer F.Cu) (net 22))
+  (segment (start 92.198 94.992) (end 92.198 98.1825) (width 0.127) (layer F.Cu) (net 22))
+  (segment (start 91.44 94.234) (end 92.198 94.992) (width 0.127) (layer F.Cu) (net 22))
   (segment (start 90.944 77.7125) (end 88.8885 77.7125) (width 0.0889) (layer F.Cu) (net 23))
   (segment (start 87.376 76.2) (end 86.36 76.2) (width 0.0889) (layer F.Cu) (net 23))
