File: pcb/usb_pmod.sch (KiCad schematic (older format))
At the start: 25 parts, among them J1 PMOD A, J2 HOST DEBUG, J3 PMOD B, J4 USB_A, J5 DEV DEBUG, J6 AU-Y1007, U1 STUSB03E, U2 STUSB03E

Commit message: Fix labels.
Connections:
- net labels removed: VBUS
- wire segments 134 -> 136
Changed lines of the file:
@@
 Wire Wire Line
 	3250 2400 3350 2400
-Wire Wire Line
-	7900 1650 7100 1650
 Connection ~ 7100 1650
 $Comp
@@
 	5850 2550 5850 2600
 Wire Wire Line
-	6850 4400 7650 4400
-Wire Wire Line
 	5850 2600 7100 2600
 Connection ~ 5850 2600
@@
 Wire Wire Line
 	5600 5350 6850 5350
-Wire Wire Line
-	8800 1950 9150 1950
 $Comp
 L power:GND #PWR015
@@
 	-1   0    0    -1
 $EndComp
-Wire Wire Line
-	8550 4600 8900 4600
 $Comp
 L power:GND #PWR016
@@
 	1    0    0    -1
 $EndComp
-Text Label 7300 4400 0    50   ~ 0
+Text Label 7600 4400 0    50   ~ 0
 H_VBUS
 Wire Wire Line
@@
 Wire Wire Line
 	7700 4800 8200 4800
-Text Label 8550 4600 0    50   ~ 0
-VBUS
 Wire Wire Line
 	6900 2050 8250 2050
@@
 Text Label 3400 2200 0    50   ~ 0
 D_VM
-Text Label 8800 1950 0    50   ~ 0
-D_VBUS
 $Comp
 L Connector:TestPoint DP1
@@
 Wire Wire Line
 	8200 4900 8900 4900
+Wire Wire Line
+	8650 1650 8650 1950
+Wire Wire Line
+	7100 1650 8650 1650
+Wire Wire Line
+	8650 1950 9150 1950
+Wire Wire Line
+	8650 4400 8650 4600
+Wire Wire Line
+	6850 4400 8650 4400
+Wire Wire Line
+	8650 4600 8900 4600
 $EndSCHEMATC
